File: electricity_hacker.kicad_sch (KiCad schematic)
At the start: 6 parts, among them SW1 SW_Push, SW2 SW_SPDT, U1 HighVoltage Module, U2 DC-DC Converter

Commit message: Add estimates
Parts:
- added D1: LED, symbol Device:LED
Connections:
- net at SW1.1, SW2.1 (A): now also D1.2 (A)
- net at BT1.2 (-), U2.2: now also D1.1 (K)
Other:
- moved on the sheet: SW2
Changed lines of the file:
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@@
 		)
+	)
+	(junction
+		(at 93.98 104.14)
+		(diameter 0)
+		(color 0 0 0 0)
+	)
+	(junction
+		(at 93.98 115.57)
+		(diameter 0)
+		(color 0 0 0 0)
 	)
 	(no_connect
-		(at 92.71 109.22)
-	)
-	(wire
-		(pts
-			(xy 66.04 115.57) (xy 101.6 115.57)
+		(at 88.9 109.22)
+	)
+	(wire
+		(pts
+			(xy 66.04 115.57) (xy 93.98 115.57)
 		)
 		(stroke
@@
 	(wire
 		(pts
+			(xy 93.98 104.14) (xy 96.52 104.14)
+		)
+		(stroke
+			(width 0)
+			(type default)
+		)
+	)
+	(wire
+		(pts
+			(xy 93.98 115.57) (xy 101.6 115.57)
+		)
+		(stroke
+			(width 0)
+			(type default)
+		)
+	)
+	(wire
+		(pts
 			(xy 154.94 109.22) (xy 154.94 113.03)
 		)
@@
 	(wire
 		(pts
-			(xy 66.04 106.68) (xy 82.55 106.68)
+			(xy 93.98 104.14) (xy 93.98 105.41)
+		)
+		(stroke
+			(width 0)
+			(type default)
+		)
+	)
+	(wire
+		(pts
+			(xy 66.04 106.68) (xy 78.74 106.68)
 		)
 		(stroke
@@
 	(wire
 		(pts
-			(xy 92.71 104.14) (xy 96.52 104.14)
+			(xy 93.98 113.03) (xy 93.98 115.57)
+		)
+		(stroke
+			(width 0)
+			(type default)
+		)
+	)
+	(wire
+		(pts
+			(xy 88.9 104.14) (xy 93.98 104.14)
 		)
 		(stroke
@@
 	(symbol
 		(lib_id "Switch:SW_SPDT")
-		(at 87.63 106.68 0)
+		(at 83.82 106.68 0)
 		(unit 1)
 		(exclude_from_sim no)
@@
 		(fields_autoplaced yes)
 		(property "Reference" "SW2"
-			(at 87.63 97.79 0)
+			(at 83.82 97.79 0)
 			(effects
 				(font
@@
 		)
 		(property "Value" "SW_SPDT"
-			(at 87.63 100.33 0)
+			(at 83.82 100.33 0)
 			(effects
 				(font
@@
 		)
 		(property "Footprint" ""
-			(at 87.63 106.68 0)
+			(at 83.82 106.68 0)
 			(effects
 				(font
@@
 		)
 		(property "Datasheet" "~"
-			(at 87.63 114.3 0)
+			(at 83.82 114.3 0)
 			(effects
 				(font
@@
 		)
 		(property "Description" "Switch, single pole double throw"
-			(at 87.63 106.68 0)
+			(at 83.82 106.68 0)
 			(effects
 				(font
@@
 					(unit 1)
 				)
+			)
+		)
+	)
+	(symbol
+		(lib_id "Device:LED")
+		(at 93.98 109.22 90)
+		(unit 1)
+		(exclude_from_sim no)
+		(in_bom yes)
+		(on_board yes)
+		(dnp no)
+		(fields_autoplaced yes)
+		(property "Reference" "D1"
+			(at 97.79 109.5374 90)
+			(effects
+				(font
+					(size 1.27 1.27)
+				)
+				(justify right)
+			)
+		)
+		(property "Value" "LED"
+			(at 97.79 112.0774 90)
+			(effects
+				(font
+					(size 1.27 1.27)
+				)
+				(justify right)
+			)
+		)
+		(property "Footprint" ""
+			(at 93.98 109.22 0)
+			(effects
+				(font
+					(size 1.27 1.27)
+				)
+				(hide yes)
+			)
+		)
+		(property "Datasheet" "~"
+			(at 93.98 109.22 0)
+			(effects
+				(font
+					(size 1.27 1.27)
+				)
+				(hide yes)
+			)
+		)
+		(property "Description" "Light emitting diode"
+			(at 93.98 109.22 0)
+			(effects
+				(font
+					(size 1.27 1.27)
+				)
+				(hide yes)
+			)
+		)
+		(property "Sim.Pins" "1=K 2=A"
+			(at 93.98 109.22 0)
+			(effects
+				(font
+					(size 1.27 1.27)
+				)
+				(hide yes)
+			)
+		)
+		(pin "1"
+		)
+		(pin "2"
+		)
+		(instances
+			(project ""
+				(path "/1b8a17c7-078e-47d4-acb4-1185cd0d34ef"
+					(reference "D1")
+					(unit 1)
+				)
